File: 6502-thing.sch (EAGLE design)
At the start: 51 parts, among them IC1 6502, IC3 555, IC5 4056N, IC6 4028N, J1 POWER_JACK, J2 CONN_20X2, J3 IO, J4 CONN_20X2, Q1 200mA/40V, Q2 200mA/40V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

Commit message: Route board.
Connections:
- net PWRIN: no longer J4.36
- net R/W: now also J4.36
Changed lines of the file:
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@@
 <?xml version="1.0" encoding="utf-8"?>
 <!DOCTYPE eagle SYSTEM "eagle.dtd">
-<eagle version="9.5.2">
+<eagle version="9.6.0">
 <drawing>
 <settings>
@@
 <pinref part="EEPROM1" gate="G$1" pin="!WE!"/>
 </segment>
+<segment>
+<wire x1="198.12" y1="114.3" x2="200.66" y2="114.3" width="0.1524" layer="91"/>
+<label x="200.66" y="114.3" size="1.27" layer="95" xref="yes"/>
+<pinref part="J4" gate="G$1" pin="36"/>
+</segment>
 </net>
 <net name="MS1" class="0">
@@
 <label x="33.02" y="-27.94" size="1.27" layer="95" rot="R90"/>
 </segment>
-<segment>
-<wire x1="198.12" y1="114.3" x2="200.66" y2="114.3" width="0.1524" layer="91"/>
-<label x="200.66" y="114.3" size="1.27" layer="95" xref="yes"/>
-<pinref part="J4" gate="G$1" pin="36"/>
-</segment>
-</net>
+</net>
