File: 6502-thing.brd (EAGLE design)
At the start: 198.1 x 150.8 mm, 56 parts, among them IC1 6502, IC3 555, IC5 4056N, IC6 4028N, J1 POWER_JACK, J2 CONN_20X2, J3 IO, J4 CONN_20X2, Q1 200mA/40V, Q2 200mA/40V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

Commit message: (liam forgot what he did in this commit)
Parts:
- removed Q5, Q6: 200mA/40V, SparkFun-DiscreteSemi:TO-92
- removed R11, R12: 10k, SparkFun-Resistors:AXIAL-0.3
- removed R13: 1k, SparkFun-Resistors:AXIAL-0.3
Connections:
- removed net EPS: Q5.1, R13.P$2
- removed net N$1: Q5.3, Q6.1
- removed net N$13: Q5.2, R12.P$2
- removed net N$7: Q6.2, R11.P$2
- net GND: no longer R13.P$1
- net MEM_EN: no longer R12.P$1
- net MS8: no longer R11.P$1
- net VCC: no longer Q6.3
Routing:
- net N$1: track 70.3 -> 0.00 mm, vias 1 -> 0
- net N$7: track 13.5 -> 0.00 mm
- net VCC: track 775.6 -> 763.6 mm
- net MEM_EN: track 195.2 -> 185.0 mm
- net EPS: track 4.07 -> 0.00 mm
- net N$13: track 3.44 -> 0.00 mm

Commit message: Move around Silkscreen a little bit.
Routing:
- net VCC: track 763.6 -> 0.00 mm, vias 4 -> 0
- net R/W: track 497.5 -> 0.00 mm, vias 9 -> 0
- net A8: track 474.4 -> 0.00 mm, vias 7 -> 0
- net A2: track 472.1 -> 0.00 mm, vias 7 -> 0
- net A6: track 466.7 -> 0.00 mm, vias 9 -> 0
- net A7: track 461.6 -> 0.00 mm, vias 6 -> 0
- net A1: track 456.6 -> 0.00 mm, vias 7 -> 0
- net A4: track 454.9 -> 0.00 mm, vias 7 -> 0
- net A3: track 446.2 -> 0.00 mm, vias 5 -> 0
- net RESET: track 440.5 -> 0.00 mm, vias 7 -> 0
- net A5: track 440.1 -> 0.00 mm, vias 8 -> 0
- net D7: track 427.0 -> 0.00 mm, vias 3 -> 0
- net D6: track 419.2 -> 0.00 mm, vias 5 -> 0
- net A13: track 410.4 -> 0.00 mm, vias 5 -> 0
- net A0: track 408.0 -> 0.00 mm, vias 8 -> 0
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Other:
- board text added: "03072020"
- board text added: "6502 board LiamCoalStudios"
- board text removed: "Build Rev 0001"
- board text removed: "LiamCoalStudios"
- board text removed: "iNsErT dAtE"

Commit message: Route board.
Parts:
- moved R21 49.9 mm to (-17.8, 101.0), turned to 90 degrees
- moved R22 31.1 mm to (-17.8, 88.3), turned to 270 degrees
- moved R5 23.6 mm to (8.26, 97.2)
- moved R24 18.8 mm to (5.08, 90.2), turned to 270 degrees
- moved MEMSEL1 16.5 mm to (16.5, 104.8)
- moved R17 16.4 mm to (8.26, 104.8)
- moved IC1 13.4 mm to (-6.35, 80.6)
- moved U$2 13.4 mm to (-32.4, 80.6)
- moved MEMORY1 11.4 mm to (40.6, 104.8)
- moved MEMORY2 10.8 mm to (64.8, 104.8)
- moved MEMORY3 10.3 mm to (88.9, 104.8)
- moved EEPROM1 9.71 mm to (113.0, 104.8)
- moved MEMORY4 6.38 mm to (40.6, 54.0)
- moved R23 5.46 mm to (8.26, 99.7), turned to 0 degrees
- moved MEMORY5 5.12 mm to (64.8, 54.0)
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Connections:
- net PWRIN: no longer J4.36
- net R/W: now also J4.36
Routing:
- net VCC: track 0.00 -> 783.5 mm, vias 0 -> 3
- net R/W: track 0.00 -> 525.6 mm, vias 0 -> 8
- net A2: track 0.00 -> 466.5 mm, vias 0 -> 5
- net A6: track 0.00 -> 455.3 mm, vias 0 -> 6
- net D7: track 0.00 -> 452.5 mm, vias 0 -> 1
- net A3: track 0.00 -> 444.3 mm, vias 0 -> 7
- net A4: track 0.00 -> 441.2 mm, vias 0 -> 6
- net D6: track 0.00 -> 432.0 mm, vias 0 -> 1
- net A5: track 0.00 -> 426.8 mm, vias 0 -> 7
- net A0: track 0.00 -> 424.9 mm, vias 0 -> 5
- net A8: track 0.00 -> 423.1 mm, vias 0 -> 7
- net A7: track 0.00 -> 421.2 mm, vias 0 -> 5
- net D5: track 0.00 -> 418.6 mm, vias 0 -> 2
- net A1: track 0.00 -> 414.9 mm, vias 0 -> 6
- net D4: track 0.00 -> 412.8 mm, vias 0 -> 2
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Other:
- board size 198.1 x 150.8 mm -> 198.1 x 163.8 mm
- board text added: "03112020"
- board text added: "Size in millimeters. (unless specified)"
- board text removed: "03072020"
